File: template/stm32_base.kicad_sch (KiCad schematic)
At the start: 41 parts, among them J1 Network Connector, J2 STDC14, SW1 SW_Push, U1 LD39050PU33R, U2 STM32G474RBT6, U3 SN65HVD230, Y1 8MHz

Commit message: telemetry-battery: update of the template according to the Template_Protocolv1.0 available in the exo-template-pcb github the 2026-10-23
Parts:
- removed C6: 100n, Capacitor_SMD:C_0402_1005Metric, symbol Device:C
- removed F1: 2A, Exocet:Fuse_Holder_Littelfuse_01530008, symbol Device:Fuse
- removed TP5: TestPoint, TestPoint:TestPoint_Keystone_5005-5009_Compact, symbol Connector:TestPoint
- removed U1: LD39050PU33R, Package_DFN_QFN:DFN-6-1EP_3x3mm_P0.95mm_EP1.7x2.6mm, symbol Exocet:LD39050PU33R
- removed U3: SN65HVD230, Package_SO:SOIC-8_3.9x4.9mm_P1.27mm, symbol Interface_CAN_LIN:SN65HVD230
- added C18: 2.2uf, Capacitor_SMD:C_01005_0402Metric, symbol Device:C
- added C19: 10uf, Capacitor_SMD:C_0805_2012Metric, symbol Device:C
- added D3: SMF28A, Diode_SMD:D_SOD-123F, symbol Device:D_Zener
- added D4, D5: SMF4L24CA, Diode_SMD:D_SOD-123F, symbol Diode:1N630xCA
- added D6: D, symbol Device:D
- added F2: 5, Exocet:Fuse_Holder_Littelfuse_01530008, symbol Device:Fuse
- added FB3: FerriteBead, Resistor_SMD:R_0805_2012Metric, symbol Device:FerriteBead
- added R6: 100, symbol Device:R
- added TP6: RED, Package_TO_SOT_SMD:SOT-23-5, symbol Connector:TestPoint
- added TP7: BLACK, symbol Connector:TestPoint
- added U1: TSR1-2450E, Converter_DCDC:Converter_DCDC_TRACO_TSR1-xxxxE_THT, symbol Converter_DCDC:TSR1-2450E
- added U3: TJA1042T-3, Package_SO:SOIC-8_3.9x4.9mm_P1.27mm, symbol Interface_CAN_LIN:TJA1042T-3
- added U4: LM3940, Package_TO_SOT_THT:TO-220-3_Vertical, symbol Exocet:LM3940
- C1: value 100n -> 470n; footprint Capacitor_SMD:C_0402_1005Metric -> Capacitor_SMD:C_0201_0603Metric; JLCPCB C1525 -> C1623
- C18: renamed from C17; value 100n -> 2.2u
- C4: value 1u -> 47u; footprint Capacitor_SMD:C_0402_1005Metric -> (none); JLCPCB C52923 -> (none)
- C5: value 1u -> 100n; JLCPCB C52923 -> (none)
- C9: footprint Capacitor_SMD:C_0402_1005Metric -> Package_SO:SOIC-8_3.9x4.9mm_P1.27mm; JLCPCB C1525 -> (none)
- H1, H2, H3, H4: value 2.7mm -> M3; footprint MountingHole:MountingHole_2.7mm_Pad -> MountingHole:MountingHole_3.2mm_M3
- R3: value 10k -> 1k; footprint Resistor_SMD:R_0402_1005Metric -> (none); JLCPCB C25744 -> (none)
- R4, R5: value 100 -> 1k
Connections:
- net +24V: now also C19.1, D3.1 (K), F2.2, TP6.1, U1.1 (Vin); no longer J1.1 (+24V)
- net +3.3V: now also C4.1, FB3.1, U3.5 (VIO), U4.3 (OUT); no longer C5.1, C7.1, C8.1, C9.1, U2.29 (VDDA)
- net +5V: now also U1.3 (Vout), U4.1 (IN); no longer C4.1, TP3.1
- net CAN_H: now also J1.3 (CAN_H), D5.2 (A2), U3.7 (CANH); no longer J1.4 (CAN_H)
- net CAN_L: now also J1.2 (CAN_L), D4.2 (A2), U3.6 (CANL); no longer J1.3 (CAN_L)
- net CAN_RX: now also U3.4 (RXD)
- net CAN_TX: now also U3.1 (TXD)
- net GND: now also C18.2, C9.1, J1.4 (GND), C18.2, C19.2, D3.2 (A), D4.1 (A1), D5.1 (A1), R6.2, TP7.1, U1.2 (GND), U3.2 (GND), U4.2 (GND); no longer C18.1, C4.2, C9.2, J1.5 (GND), SW1.2
- net T_NRST: now also C18.1, D6.2 (A); no longer C18.2, SW1.1
- net at R3.1: now also U3.8 (STB)
- new net: C7.1, C8.1, FB3.2, U2.29 (VDDA)
- new net: C18.1, D6.1 (K), SW1.1
- new net: R6.1, SW1.2
- new net: F2.1, J1.1 (+24V)
- new net: C4.2, C5.1
- new net 5V VDC: C9.2, TP3.1, U3.3 (VCC)
- no-connect marks 42 -> 40
Other:
- note added: "Voltage Regulator 1"
- note added: "Voltage Regulator 2"
- note removed: "Voltage Regulator"
- company: (none) -> Exocet Polytechnique Montréal
- moved on the sheet: C18, C2, C3, C7, C8, SW1, TP1, TP3
