File: telemetry-battery-pcb/stm32_base.kicad_sch (KiCad schematic)
At the start: 0 parts

Commit message: telemetry-battery: update of the template according to the Template_Protocolv1.0 available in the exo-template-pcb github the 2026-10-23
Parts:
- added C1, C10, C11, C12, C13, C17, C3, C6, C9: 100n, Capacitor_SMD:C_0402_1005Metric, symbol Device:C
- added C14: 4.7u, Capacitor_SMD:C_0402_1005Metric, symbol Device:C
- added C15, C16: 30p, Capacitor_SMD:C_0603_1608Metric, symbol Device:C
- added C2, C4, C5, C8: 1u, Capacitor_SMD:C_0402_1005Metric, symbol Device:C
- added C7: 10n, Capacitor_SMD:C_0402_1005Metric, symbol Device:C
- added D1: GREEN, Exocet:LED_0805_2012Metric_With_Annotations, symbol Device:LED
- added D2: YELLOW, Exocet:LED_0805_2012Metric_With_Annotations, symbol Device:LED
- added F1: 2A, Exocet:Fuse_Holder_Littelfuse_01530008, symbol Device:Fuse
- added H1, H2, H3, H4: 2.7mm, MountingHole:MountingHole_2.7mm_Pad, symbol Mechanical:MountingHole_Pad
- added J1: Network Connector, Connector_Molex:Molex_SPOX_5268-05A_1x05_P2.50mm_Horizontal, symbol Exocet:Network_Connector
- added J2: STDC14, Connector_PinHeader_1.27mm:PinHeader_2x07_P1.27mm_Vertical_SMD, symbol Connector:Conn_ST_STDC14
- added R1, R3: 10k, Resistor_SMD:R_0402_1005Metric, symbol Device:R
- added R2: 47, Resistor_SMD:R_0603_1608Metric, symbol Device:R
- added R4, R5: 100, Resistor_SMD:R_0402_1005Metric, symbol Device:R
- added SW1: SW_Push, Button_Switch_THT:SW_PUSH_6mm, symbol Switch:SW_Push
- added TP1, TP2, TP3, TP4, TP5: TestPoint, TestPoint:TestPoint_Keystone_5005-5009_Compact, symbol Connector:TestPoint
- added U1: LD39050PU33R, Package_DFN_QFN:DFN-6-1EP_3x3mm_P0.95mm_EP1.7x2.6mm, symbol Exocet:LD39050PU33R
- added U2: STM32G474RBT6, Package_QFP:LQFP-64_10x10mm_P0.5mm, symbol MCU_ST_STM32G4:STM32G474RBTx
- added U3: SN65HVD230, Package_SO:SOIC-8_3.9x4.9mm_P1.27mm, symbol Interface_CAN_LIN:SN65HVD230
- added Y1: 8MHz, Exocet:Crystal_SMD_HC49-SD, symbol Exocet:HSE_Oscillator
Connections:
- new net: R2.1, U2.51 (PA15)
- new net: R1.1, U2.61 (PB8)
- new net: R3.1, U3.8 (Rs)
- new net: D1.2 (A), R4.2
- new net: D2.2 (A), R5.2
- new net: F1.1, J1.2 (+5V)
- new net +24V: J1.1 (+24V)
- new net +3.3V: C10.1, C11.1, C12.1, C13.1, C14.1, C2.2, C3.2, C5.1, C6.1, C7.1, C8.1, C9.1, J2.3 (VCC), R4.1, TP5.1, U1.4 (V_{out}), U2.1 (VBAT), U2.16 (VDD), U2.28 (VREF+), U2.29 (VDDA), U2.32 (VDD), U2.48 (VDD), U2.64 (VDD), U3.3 (VCC)
- new net +5V: C1.1, C4.1, F1.2, TP3.1, U1.1 (EN), U1.6 (V_{in})
- new net CAN_H: J1.4 (CAN_H), U3.7 (CANH)
- new net CAN_L: J1.3 (CAN_L), U3.6 (CANL)
- new net CAN_RX: TP2.1, U2.45 (PA11), U3.4 (R)
- new net CAN_TX: TP4.1, U2.46 (PA12), U3.1 (D)
- new net GND: C1.2, C10.2, C11.2, C12.2, C13.2, C14.2, C15.2, C16.2, C17.1, C2.1, C3.1, C4.2, C5.2, C6.2, C7.2, C8.2, C9.2, D1.1 (K), D2.1 (K), H1.1, H2.1, H3.1, H4.1, J1.5 (GND), J2.11 (GNDDetect), J2.5 (GND), J2.7 (GND), R1.2, R3.2, SW1.2, TP1.1, U1.2 (GND), U1.7 (GND), U2.15 (VSS), U2.27 (VSSA), U2.31 (VSS), U2.47 (VSS), U2.63 (VSS), U3.2 (GND)
- new net OSC_IN: C15.1, U2.5 (PF0), Y1.1
- new net OSC_OUT: C16.1, U2.6 (PF1), Y1.2
- new net STATUS_LED: R5.1, U2.8 (PC0)
- new net T_JCLK/T_SWCLK: J2.6 (JCLK/SWCLK), U2.50 (PA14)
- new net T_JTDI: J2.10 (JTDI/NC), R2.2
- new net T_JTDO/T_SWO: J2.8 (JTDO/SWO), U2.56 (PB3)
- new net T_JTMS/T_SWDIO: J2.4 (JTMS/SWDIO), U2.49 (PA13)
- new net T_NRST: C17.2, J2.12 (~{RST}), SW1.1, U2.7 (PG10)
- new net T_VCP_RX: J2.13 (VCP_RX), U2.17 (PA3)
- new net T_VCP_TX: J2.14 (VCP_TX), U2.14 (PA2)
- no-connect marks 0 -> 42
Other:
- note added: "CAN Tranceiver"
- note added: "Mounting Holes"
- note added: "Network Connector"
- note added: "Oscillator"
- note added: "Reset Button"
- note added: "STLink Connector"
- note added: "STM32 MCU"
- note added: "Status LEDs"
- note added: "Test Points"
- note added: "Voltage Regulator"
- title: (none) -> STM32 Base Layout

Commit message: telemetry-battery-pcb: update of the schematic with the new stm32 Base Model including removing the 24V converter and switch and associated devices (PGOOD).
Parts:
- removed C6: 100n, Capacitor_SMD:C_0402_1005Metric, symbol Device:C
- removed F1: 2A, Exocet:Fuse_Holder_Littelfuse_01530008, symbol Device:Fuse
- removed TP5: TestPoint, TestPoint:TestPoint_Keystone_5005-5009_Compact, symbol Connector:TestPoint
- removed U1: LD39050PU33R, Package_DFN_QFN:DFN-6-1EP_3x3mm_P0.95mm_EP1.7x2.6mm, symbol Exocet:LD39050PU33R
- removed U3: SN65HVD230, Package_SO:SOIC-8_3.9x4.9mm_P1.27mm, symbol Interface_CAN_LIN:SN65HVD230
- added C18: 2.2uf, Capacitor_SMD:C_01005_0402Metric, symbol Device:C
- added C19: 10uf, Capacitor_SMD:C_0805_2012Metric, symbol Device:C
- added D3: SMF28A, Diode_SMD:D_SOD-123F, symbol Device:D_Zener
- added D4, D5: SMF4L24CA, Diode_SMD:D_SOD-123F, symbol Diode:1N630xCA
- added D6: D, symbol Device:D
- added F2: 5, Exocet:Fuse_Holder_Littelfuse_01530008, symbol Device:Fuse
- added FB3: FerriteBead, Resistor_SMD:R_0805_2012Metric, symbol Device:FerriteBead
- added R6: 100, symbol Device:R
- added TP6: RED, Package_TO_SOT_SMD:SOT-23-5, symbol Connector:TestPoint
- added TP7: BLACK, symbol Connector:TestPoint
- added U1: TSR1-2450E, Converter_DCDC:Converter_DCDC_TRACO_TSR1-xxxxE_THT, symbol Converter_DCDC:TSR1-2450E
- added U3: TJA1042T-3, Package_SO:SOIC-8_3.9x4.9mm_P1.27mm, symbol Interface_CAN_LIN:TJA1042T-3
- added U4: LM3940, Package_TO_SOT_THT:TO-220-3_Vertical, symbol Exocet:LM3940
- C1: value 100n -> 470n; footprint Capacitor_SMD:C_0402_1005Metric -> Capacitor_SMD:C_0201_0603Metric; JLCPCB C1525 -> C1623
- C18: renamed from C17; value 100n -> 2.2u
- C4: value 1u -> 47u; footprint Capacitor_SMD:C_0402_1005Metric -> (none); JLCPCB C52923 -> (none)
- C5: value 1u -> 100n; JLCPCB C52923 -> (none)
- C9: footprint Capacitor_SMD:C_0402_1005Metric -> Package_SO:SOIC-8_3.9x4.9mm_P1.27mm; JLCPCB C1525 -> (none)
- H1, H2, H3, H4: value 2.7mm -> M3; footprint MountingHole:MountingHole_2.7mm_Pad -> MountingHole:MountingHole_3.2mm_M3
- R3: value 10k -> 1k; footprint Resistor_SMD:R_0402_1005Metric -> (none); JLCPCB C25744 -> (none)
- R4, R5: value 100 -> 1k
Connections:
- net +24V: now also C19.1, D3.1 (K), F2.2, TP6.1, U1.1 (Vin); no longer J1.1 (+24V)
- net +3.3V: now also C4.1, FB3.1, U3.5 (VIO), U4.3 (OUT); no longer C5.1, C7.1, C8.1, C9.1, U2.29 (VDDA)
- net +5V: now also U1.3 (Vout), U4.1 (IN); no longer C4.1, TP3.1
- net CAN_H: now also J1.3 (CAN_H), D5.2 (A2), U3.7 (CANH); no longer J1.4 (CAN_H)
- net CAN_L: now also J1.2 (CAN_L), D4.2 (A2), U3.6 (CANL); no longer J1.3 (CAN_L)
- net CAN_RX: now also U3.4 (RXD)
- net CAN_TX: now also U3.1 (TXD)
- net GND: now also C18.2, C9.1, J1.4 (GND), C18.2, C19.2, D3.2 (A), D4.1 (A1), D5.1 (A1), R6.2, TP7.1, U1.2 (GND), U3.2 (GND), U4.2 (GND); no longer C18.1, C4.2, C9.2, J1.5 (GND), SW1.2
- net T_NRST: now also C18.1, D6.2 (A); no longer C18.2, SW1.1
- net at R3.1: now also U3.8 (STB)
- new net: C7.1, C8.1, FB3.2, U2.29 (VDDA)
- new net: C18.1, D6.1 (K), SW1.1
- new net: R6.1, SW1.2
- new net: F2.1, J1.1 (+24V)
- new net: C4.2, C5.1
- new net 5V VDC: C9.2, TP3.1, U3.3 (VCC)
- no-connect marks 42 -> 40
Other:
- note added: "Voltage Regulator 1"
- note added: "Voltage Regulator 2"
- note removed: "Voltage Regulator"
- company: (none) -> Exocet Polytechnique Montréal
- moved on the sheet: C18, C2, C3, C7, C8, SW1, TP1, TP3
